File: hardware/apple-ice.sch (KiCad schematic (older format))
At the start: 34 parts, among them J1 TO_SP_DRIVE, P1 A2Bus-apple2, U1 ICE40HX1K-TQ144, U10 SN74LVC8T245PW, U2 SN74LVC8T245PW, U3 SN74LVC8T245PW, U4 SN74LVC8T245PW, U5 SN74LVC8T245PW, U6 MCP1703A-3302_SOT223, U7 MCP1703A-1202_SOT223, U8 W25Q16JVSS, U9 SN74LVC8T245PW

Commit message: FPGA programming and power
Reorginize schematic
Add more footprints and symbols

Signed-off-by: Rangel Ivanov <rangelivanov88@gmail.com>
Parts:
- added C? (x10): 100n, symbol apple-ice:C_Small
- added C? (x5): 1u, symbol apple-ice:C_Small
- added C?: 100n, apple-ice:C_0603_1608Metric_Pad1.08x0.95mm_HandSolder, symbol apple-ice:C_Small
- added D?: 1N5819, apple-ice:D_SOD-123, symbol apple-ice:1N5819
- added D? (x3): LED, symbol apple-ice:LED
- added J?: SPI_FLASH_PROG, symbol apple-ice:Conn_02x05_Odd_Even
- added J?: USB_B_Micro, symbol apple-ice:USB_B_Micro
- added JP?: J_USB_5V, symbol apple-ice:Jumper_NO_Small
- added R? (x2): 10, symbol apple-ice:R_Small
- added R? (x7): 10k, symbol apple-ice:R_Small
- added R? (x3): 2k2, symbol apple-ice:R_Small
- added R? (x3): 22, symbol apple-ice:R_Small
- added R?: 1k5, symbol apple-ice:R_Small
- added SW? (x3): SW_Push, symbol apple-ice:SW_Push
- added X?: ECS-2520MV-xxx-xx, apple-ice:Oscillator_SMD_ECS_2520MV-xxx-xx-4Pin_2.5x2.0mm, symbol apple-ice:ECS-2520MV-xxx-xx
- C?: renamed from C1; footprint (none) -> apple-ice:C_0603_1608Metric_Pad1.08x0.95mm_HandSolder
- C?: renamed from C3; footprint (none) -> apple-ice:C_0603_1608Metric_Pad1.08x0.95mm_HandSolder
- C?: renamed from C2; footprint (none) -> apple-ice:C_0603_1608Metric_Pad1.08x0.95mm_HandSolder
- C?: renamed from C4; footprint (none) -> apple-ice:C_0603_1608Metric_Pad1.08x0.95mm_HandSolder
- C?: renamed from C5; footprint (none) -> apple-ice:C_0603_1608Metric_Pad1.08x0.95mm_HandSolder
- C?: renamed from C6; footprint (none) -> apple-ice:C_0603_1608Metric_Pad1.08x0.95mm_HandSolder
- C? (x10): footprint (none) -> apple-ice:C_0603_1608Metric_Pad1.08x0.95mm_HandSolder
- R?: renamed from R2; footprint (none) -> apple-ice:R_0603_1608Metric_Pad0.98x0.95mm_HandSolder
- R?: renamed from R4; footprint (none) -> apple-ice:R_0603_1608Metric_Pad0.98x0.95mm_HandSolder
- R?: renamed from R1; footprint (none) -> apple-ice:R_0603_1608Metric_Pad0.98x0.95mm_HandSolder
- R?: renamed from R6; footprint (none) -> apple-ice:R_0603_1608Metric_Pad0.98x0.95mm_HandSolder
- R?: renamed from R5; footprint (none) -> apple-ice:R_0603_1608Metric_Pad0.98x0.95mm_HandSolder
- R?: renamed from R3; footprint (none) -> apple-ice:R_0603_1608Metric_Pad0.98x0.95mm_HandSolder
- renumbered J1 to J?, P1 to P?, U1 to U?, U8 to U?, U2 to U?, U4 to U?, U7 to U?, U5 to U?, U6 to U?, U3 to U?, U10 to U?, U9 to U?
Connections:
- net 1.2V is gone; now on net +1V2: C?.1, U?.3 (VO)
- net 12V is gone; now on net +12V: J?.13 (Pin_13), J?.15 (Pin_15)
- net +5V: now also U?.23 (VCC(B)), U?.24 (VCC(B)), C?.2, JP?.1; no longer U?.1 (VCC(A))
- net -12V: now also P?.33 (-12V)
- net GND: now also P?.26 (GND), U?.103 (GND), U?.13 (GND), U?.132 (GND), U?.14 (GND), U?.140 (GND), U?.4 (GND), U?.5 (GND), U?.59 (GND), U?.69 (GND), U?.86 (GND), C?.1, C?.2, C?.2, C?.2, C?.2, C?.2, C?.2, C?.2, C?.2, C?.2, C?.2, C?.2, C?.2, C?.2, C?.2, J?.2 (Pin_2), J?.5 (GND), J?.6 (Shield), R?.1, R?.1, R?.2, SW?.1, SW?.2, SW?.2, X?.2 (GND)
- net ~INH: now also U?.38 (IOB_25), U?.4 (A2); no longer U?.39 (IOB_26), U?.5 (A3)
- net ~IRQ: now also U?.39 (IOB_26), U?.5 (A3); no longer U?.4 (A2), U?.41 (IOB_27)
- net ~NMI: now also U?.41 (IOB_27), U?.6 (A4); no longer U?.3 (A1), U?.42 (IOB_28)
- net ~RDY: now also U?.3 (A1), U?.37 (IOB_24); no longer U?.38 (IOB_25), U?.6 (A4)
- net +3.3V: now reaches U?.123 (VCCIO_0), U?.133 (VCCIO_0)
- net +3.3V: now also C?.1, C?.2, C?.2, C?.2, C?.2, C?.2, C?.2, R?.1, R?.1, R?.1, U?.1 (VCC(A)), U?.1 (VCC(A)), U?.1 (VCC(A)), U?.1 (VCC(A)), U?.1 (VCC(A)), U?.1 (VCC(A)), U?.100 (VCCIO_1), U?.3 (VO), U?.30 (VCCIO_3), U?.46 (VCCIO_2), U?.57 (VCCIO_2), U?.6 (VCCIO_3), U?.72 (VCC_SPI), U?.8 (VCC), U?.89 (VCCIO_1), C?.1, C?.1, C?.1, C?.1, C?.1, C?.1, C?.1, C?.1, C?.1, C?.1, C?.1, D?.2 (A), R?.1, R?.1, R?.1, R?.1, R?.1, R?.1, R?.1, R?.1, R?.1
- net ~FLASH_WP(~IO3): now reaches U?.78 (IOR_52)
- net ~FLASH_WP(~IO3): now also U?.3 (IO2), R?.2
- net ~FLASH_HOLD(~IO4): now reaches U?.79 (IOR_53)
- net ~FLASH_HOLD(~IO4): now also U?.7 (IO3), R?.2
- net BTN1: now reaches U?.80 (IOR_54)
- net BTN1: now also R?.2, SW?.1
- net BTN2: now reaches U?.81 (IOR_55)
- net BTN2: now also R?.2, SW?.1
- net LED1: now reaches U?.87 (IOR_56)
- net LED1: now also D?.2 (A)
- net LED2: now reaches U?.88 (IOR_57)
- net LED2: now also D?.2 (A)
- net USB_P: now reaches U?.90 (IOR_58)
- net USB_P: now also R?.1
- net USB_N: now reaches U?.91 (IOR_59)
- net USB_N: now also R?.1
- net 16Mhz: now reaches U?.93 (IOR_60_GBIN3)
- net 16Mhz: now also R?.1
- net USB_PU: now reaches U?.95 (IOR_62)
- net USB_PU: now also R?.2
- net at R?.2, U?.22 (~OE): now also U?.42 (IOB_28); no longer U?.37 (IOB_24)
- net at U?.108 (VPP_2V5): now also D?.1 (K)
- net +1V2: now reaches U?.111 (VCC), U?.27 (VCC), U?.51 (VCC), U?.92 (VCC)
- net +1V2: now also U?.36 (VCCPLL), C?.1, C?.1, C?.1, C?.1
- net at U?.35 (GNDPLL): now also C?.2
- net iCE40_CDONE: now reaches U?.65 (CDONE)
- net iCE40_CDONE: now also D?.2 (A), J?.5 (Pin_5), R?.2
- net ~iCE40_CRESET: now reaches U?.66 (~CRESET_B)
- net ~iCE40_CRESET: now also J?.6 (Pin_6), R?.2, SW?.2
- net iC40_SDO: now reaches U?.67 (IOB_44_SDO)
- net iC40_SDO: now also U?.2 (DO(IO1)), J?.8 (Pin_8)
- net iC40_SDI: now reaches U?.68 (IOB_45_SDI)
- net iC40_SDI: now also U?.5 (DI(IO0)), J?.7 (Pin_7)
- net iCE40_SCK: now reaches U?.70 (IOB_46_SCK)
- net iCE40_SCK: now also U?.6 (CLK), J?.9 (Pin_9)
- net ~iCE40_CS: now reaches U?.71 (IOB_47_SS)
- net ~iCE40_CS: now also U?.1 (~CS), J?.10 (Pin_10), R?.2
- net at U?.18 (B4): now also P?.29 (~NMI); no longer P?.21 (~RDY)
- net at U?.19 (B3): now also P?.30 (~IRQ); no longer P?.32 (~INH)
- net at U?.20 (B2): now also P?.32 (~INH); no longer P?.30 (~IRQ)
- net at U?.21 (B1): now also P?.21 (~RDY); no longer P?.29 (~NMI)
- net +12V: now reaches P?.50 (+12V)
- removed net 3.3V: C?.1, C?.2, C?.2, C?.2, C?.2, C?.2, C?.2, R?.1, R?.1, R?.1, U?.1 (VCC(A)), U?.1 (VCC(A)), U?.1 (VCC(A)), U?.1 (VCC(A)), U?.1 (VCC(A)), U?.23 (VCC(B)), U?.24 (VCC(B)), U?.3 (VO)
- new net: J?.1 (VBUS), JP?.2
- new net: R?.2, X?.1 (Tri-State)
- new net: R?.2, X?.3 (OUT)
- new net: R?.2, X?.4 (VDD)
- new net: D?.1 (K), R?.1
- new net: D?.1 (K), R?.2 (x2)
- new net: J?.2 (D-), R?.2
- new net: J?.3 (D+), R?.1, R?.2
- no-connect marks 19 -> 25
Other:
- moved on the sheet: C?, J?, P?, R?, U?, U?A, U?B, U?C, U?D, U?E

Commit message: Begin initial placement and routing
Signed-off-by: Rangel Ivanov <rangelivanov88@gmail.com>
Parts:
- C11, C12, C13, C16, C21, C22, C23, C24, C26, C27, C28, C29, C30, C31, C32: renamed from C?; footprint (none) -> apple-ice:C_0603_1608Metric_Pad1.08x0.95mm_HandSolder
- D1, D2, D3: renamed from D?; footprint (none) -> apple-ice:LED_0603_1608Metric
- J2: renamed from J?; footprint (none) -> apple-ice:USB_Micro-B_Molex-105017-0001
- J3: renamed from J?; footprint (none) -> apple-ice:IDC-Header_2x05_P2.54mm_Vertical
- JP1: renamed from JP?; footprint (none) -> apple-ice:C_0603_1608Metric_Pad1.08x0.95mm_HandSolder
- R10, R11, R12, R13, R14, R15, R16, R17, R18, R19, R20, R21, R22, R7, R8, R9: renamed from R?; footprint (none) -> apple-ice:R_0603_1608Metric_Pad0.98x0.95mm_HandSolder
- SW1, SW2, SW3: renamed from SW?; footprint (none) -> apple-ice:SW_SPST_B3S-1000
- gave numbers to parts that had none: 37
Connections:
- net D0: now also U5.21 (B1); no longer U5.14 (B8)
- net D0_33: now also U5.3 (A1); no longer U5.10 (A8)
- net D1: now also U5.20 (B2); no longer U5.15 (B7)
- net D1_33: now also U5.4 (A2); no longer U5.9 (A7)
- net D2: now also U5.19 (B3); no longer U5.16 (B6)
- net D2_33: now also U5.5 (A3); no longer U5.8 (A6)
- net D3: now also U5.18 (B4); no longer U5.17 (B5)
- net D3_33: now also U5.6 (A4); no longer U5.7 (A5)
- net D4: now also U5.17 (B5); no longer U5.18 (B4)
- net D4_33: now also U5.7 (A5); no longer U5.6 (A4)
- net D5: now also U5.16 (B6); no longer U5.19 (B3)
- net D5_33: now also U5.8 (A6); no longer U5.5 (A3)
- net D6: now also U5.15 (B7); no longer U5.20 (B2)
- net D6_33: now also U5.9 (A7); no longer U5.4 (A2)
- net D7: now also U5.14 (B8); no longer U5.21 (B1)
- net D7_33: now also U5.10 (A8); no longer U5.3 (A1)
- net 7M_33: now reaches U6.43 (IOB_29)
- net 7M_33: now also U2.10 (A8); no longer U2.3 (A1)
- net Q3_33: now reaches U6.44 (IOB_30)
- net Q3_33: now also U2.9 (A7); no longer U2.4 (A2)
- net PHI0_33: now reaches U6.45 (IOB_31)
- net PHI0_33: now also U2.8 (A6); no longer U2.5 (A3)
- net ~DEVSEL_33: now reaches U2.6 (A4)
- net ~DEVSEL_33: now also U6.48 (IOB_33); no longer U6.47 (IOB_32)
- net ~RES_33: now reaches U2.7 (A5)
- net ~RES_33: now also U6.47 (IOB_32); no longer U6.48 (IOB_33)
- net ~IOSTROBE_33: now reaches U6.49 (IOB_35_GBIN5)
- net ~IOSTROBE_33: now also U2.5 (A3); no longer U2.8 (A6)
- net ~IOSEL_33: now reaches U6.50 (IOB_36_GBIN4)
- net ~IOSEL_33: now also U2.4 (A2); no longer U2.9 (A7)
- net RW_33: now reaches U6.52 (IOB_34)
- net RW_33: now also U2.3 (A1); no longer U2.10 (A8)
- net 7M: now reaches P1.36 (7M), U2.14 (B8)
- net PHI0: now reaches P1.40 (PHI0), U2.16 (B6)
- net ~RES: now reaches P1.31 (~RES), U2.17 (B5)
- net ~DEVSEL: now reaches P1.41 (~DEVSEL), U2.18 (B4)
- net ~IOSTROBE: now reaches P1.20 (~IOSTRB), U2.19 (B3)
- net ~IOSEL: now reaches P1.01 (~IOSEL), U2.20 (B2)
- net Q3: now reaches P1.37 (Q3), R1.2

Commit message: Initial placement V2
Signed-off-by: Rangel Ivanov <rangelivanov88@gmail.com>
Connections:
- net PH0: now also U6.112 (IOT_73); no longer U6.58 (IOB_38)
- net PH1: now also U6.113 (IOT_74); no longer U6.60 (IOB_39)
- net PH2: now also U6.114 (IOT_75); no longer U6.61 (IOB_40)
- net PH3: now also U6.115 (IOT_76); no longer U6.62 (IOB_41)
- net RDDATA_33: now also U6.120 (IOT_81); no longer U6.75 (IOR_50)
- net SEL: now also U6.117 (IOT_78); no longer U6.64 (IOB_43_CBSEL1)
- net SENSE_33: now also U6.121 (IOT_82); no longer U6.76 (IOR_51)
- net WRDATA: now also U6.119 (IOT_80); no longer U6.74 (IOR_49)
- net ~ENABLE: now also U6.118 (IOT_79); no longer U6.73 (IOR_48)
- net ~WREQ: now also U6.116 (IOT_77); no longer U6.63 (IOB_42_CBSEL0)
- no-connect marks 25 -> 29
Changed lines of the file:
@@
 L apple-ice:GND #PWR0107
 U 1 1 60AB624A
-P 4500 6550
-F 0 "#PWR0107" H 4500 6300 50  0001 C CNN
+P 4500 6600
+F 0 "#PWR0107" H 4500 6350 50  0001 C CNN
 F 1 "GND" H 4600 6600 50  0000 C CNN
-F 2 "" H 4500 6550 50  0001 C CNN
-F 3 "" H 4500 6550 50  0001 C CNN
-	1    4500 6550
+F 2 "" H 4500 6600 50  0001 C CNN
+F 3 "" H 4500 6600 50  0001 C CNN
+	1    4500 6600
 	1    0    0    -1
 $EndComp
@@
 Wire Wire Line
 	5850 4000 5600 4000
-Wire Wire Line
-	6350 4850 6750 4850
-Wire Wire Line
-	6350 4750 6700 4750
-Wire Wire Line
-	6350 4650 6650 4650
-Wire Wire Line
-	6500 2450 6850 2450
-Wire Wire Line
-	6350 4350 6500 4350
 NoConn ~ 5500 4550
 Wire Wire Line
-	6350 4950 6800 4950
-Wire Wire Line
 	6350 5250 6800 5250
 Wire Wire Line
@@
 	1    0    0    -1
 $EndComp
-Text Label 9750 4950 0    50   ~ 0
-RDDATA_33
-Text Label 9750 5050 0    50   ~ 0
-SENSE_33
-Text Label 9750 4750 0    50   ~ 0
-~ENABLE
-Text Label 9750 4850 0    50   ~ 0
-WRDATA
 Wire Wire Line
 	5550 2050 5100 2050
@@
 L apple-ice:GND #PWR0137
 U 1 1 639D5C60
-P 4500 8700
-F 0 "#PWR0137" H 4500 8450 50  0001 C CNN
-F 1 "GND" H 4650 8650 50  0000 C CNN
-F 2 "" H 4500 8700 50  0001 C CNN
-F 3 "" H 4500 8700 50  0001 C CNN
-	1    4500 8700
+P 4500 8750
+F 0 "#PWR0137" H 4500 8500 50  0001 C CNN
+F 1 "GND" H 4650 8700 50  0000 C CNN
+F 2 "" H 4500 8750 50  0001 C CNN
+F 3 "" H 4500 8750 50  0001 C CNN
+	1    4500 8750
 	1    0    0    -1
 $EndComp
@@
 L apple-ice:GND #PWR0142
 U 1 1 65399DB8
-P 4500 2350
-F 0 "#PWR0142" H 4500 2100 50  0001 C CNN
-F 1 "GND" H 4505 2177 50  0000 C CNN
-F 2 "" H 4500 2350 50  0001 C CNN
-F 3 "" H 4500 2350 50  0001 C CNN
-	1    4500 2350
+P 4500 2400
+F 0 "#PWR0142" H 4500 2150 50  0001 C CNN
+F 1 "GND" H 4505 2227 50  0000 C CNN
+F 2 "" H 4500 2400 50  0001 C CNN
+F 3 "" H 4500 2400 50  0001 C CNN
+	1    4500 2400
 	1    0    0    -1
 $EndComp
@@
 	5550 1950 5550 1900
 Wire Wire Line
-	6350 4550 6600 4550
-Wire Wire Line
-	6350 4450 6550 4450
-Wire Wire Line
-	6500 2450 6500 4350
-Wire Wire Line
-	6550 4450 6550 2550
-Wire Wire Line
-	6550 2550 6850 2550
-Wire Wire Line
-	6600 4550 6600 2650
-Wire Wire Line
-	6600 2650 6850 2650
-Wire Wire Line
-	6650 4650 6650 2750
-Wire Wire Line
-	6650 2750 6850 2750
-Wire Wire Line
-	6700 4750 6700 2850
-Wire Wire Line
-	6700 2850 6850 2850
-Wire Wire Line
-	6750 4850 6750 2950
-Wire Wire Line
-	6750 2950 6850 2950
-Wire Wire Line
 	6850 2350 6500 2350
 Text Label 6500 2350 0    50   ~ 0
@@
 	-1   0    0    -1
 $EndComp
-Wire Wire Line
-	6800 4950 6800 4750
-Wire Wire Line
-	6800 4750 10500 4750
-Wire Wire Line
-	6900 5150 6900 4850
-Wire Wire Line
-	6900 4850 10500 4850
-Wire Wire Line
-	6350 5150 6900 5150
-Wire Wire Line
-	9650 6250 9650 4950
-Wire Wire Line
-	9650 4950 10500 4950
-Wire Wire Line
-	9750 6350 9750 5050
-Wire Wire Line
-	9750 5050 10500 5050
 Connection ~ 7200 6350
 Wire Wire Line
@@
 P 4400 9000
 F 0 "#PWR0156" H 4400 8850 50  0001 C CNN
-F 1 "+5V" H 4400 9150 50  0000 C CNN
+F 1 "+5V" H 4300 9050 50  0000 C CNN
 F 2 "" H 4400 9000 50  0001 C CNN
 F 3 "" H 4400 9000 50  0001 C CNN
@@
 P 4600 9000
 F 0 "#PWR0162" H 4600 8850 50  0001 C CNN
-F 1 "+3.3V" H 4600 9150 50  0000 C CNN
+F 1 "+3.3V" H 4750 9050 50  0000 C CNN
 F 2 "" H 4600 9000 50  0001 C CNN
 F 3 "" H 4600 9000 50  0001 C CNN
@@
 	11200 8750 11450 8750
 Connection ~ 11450 9750
-$Comp
-L apple-ice:C_Small C25
-U 1 1 6873492D
-P 11550 8750
-F 0 "C25" V 11600 8850 50  0000 L CNN
-F 1 "100n" V 11600 8500 50  0000 L CNN
-F 2 "apple-ice:C_0603_1608Metric_Pad1.08x0.95mm_HandSolder" H 11550 8750 50  0001 C CNN
-F 3 "~" H 11550 8750 50  0001 C CNN
-	1    11550 8750
-	0    -1   -1   0
-$EndComp
-Wire Wire Line
-	11650 8750 11950 8750
 Wire Wire Line
 	11850 9150 11950 9150
-Wire Wire Line
-	11950 9150 11950 9050
-Wire Wire Line
-	11950 8750 11950 8850
 $Comp
 L apple-ice:R_Small R11
@@
 Connection ~ 15250 5000
 $Comp
-L apple-ice:Jumper_NO_Small JP1
-U 1 1 60C25D7C
-P 11950 8950
-F 0 "JP1" V 11904 8998 50  0000 L CNN
-F 1 "J_USB_5V" V 12000 9000 50  0000 L CNN
-F 2 "apple-ice:C_0603_1608Metric_Pad1.08x0.95mm_HandSolder" H 11950 8950 50  0001 C CNN
-F 3 "~" H 11950 8950 50  0001 C CNN
-	1    11950 8950
-	0    1    1    0
-$EndComp
-Wire Wire Line
-	11950 8750 11950 8550
-Connection ~ 11950 8750
-$Comp
-L apple-ice:+5V #PWR0190
-U 1 1 60D920DD
-P 11950 8550
-F 0 "#PWR0190" H 11950 8400 50  0001 C CNN
-F 1 "+5V" H 11965 8723 50  0000 C CNN
-F 2 "" H 11950 8550 50  0001 C CNN
-F 3 "" H 11950 8550 50  0001 C CNN
-	1    11950 8550
-	1    0    0    -1
-$EndComp
-$Comp
 L apple-ice:R_Small R10
 U 1 1 689D4753
@@
 Text Label 5600 3250 2    50   ~ 0
 ~IOSTROBE_33
-Wire Bus Line
-	3700 9250 3700 10150
-Wire Bus Line
-	1300 5050 1300 9050
-Wire Bus Line
-	5500 5350 5500 10150
-Wire Bus Line
-	3650 4250 3650 8000
 Text Label 6200 2250 2    50   ~ 0
 RW_33
@@
 Text Label 6200 1550 2    50   ~ 0
 7M_33
+Wire Wire Line
+	4500 6550 4500 6600
+Wire Wire Line
+	4500 8700 4500 8750
+Wire Wire Line
+	4500 2350 4500 2400
+Wire Wire Line
+	11950 9150 11950 9050
+$Comp
+L apple-ice:+5V #PWR0190
+U 1 1 60D920DD
+P 11950 8550
+F 0 "#PWR0190" H 11950 8400 50  0001 C CNN
+F 1 "+5V" H 11965 8723 50  0000 C CNN
+F 2 "" H 11950 8550 50  0001 C CNN
+F 3 "" H 11950 8550 50  0001 C CNN
+	1    11950 8550
+	1    0    0    -1
+$EndComp
+$Comp
+L apple-ice:Jumper_NO_Small JP1
+U 1 1 60C25D7C
+P 11950 8950
+F 0 "JP1" V 11904 8998 50  0000 L CNN
+F 1 "J_USB_5V" V 12000 9000 50  0000 L CNN
+F 2 "apple-ice:C_0603_1608Metric_Pad1.08x0.95mm_HandSolder" H 11950 8950 50  0001 C CNN
+F 3 "~" H 11950 8950 50  0001 C CNN
+	1    11950 8950
+	0    1    1    0
+$EndComp
+Wire Wire Line
+	11650 8750 11950 8750
+Wire Wire Line
+	11950 8750 11950 8550
+$Comp
+L apple-ice:C_Small C25
+U 1 1 6873492D
+P 11550 8750
+F 0 "C25" V 11600 8850 50  0000 L CNN
+F 1 "100n" V 11600 8500 50  0000 L CNN
+F 2 "apple-ice:C_0603_1608Metric_Pad1.08x0.95mm_HandSolder" H 11550 8750 50  0001 C CNN
+F 3 "~" H 11550 8750 50  0001 C CNN
+	1    11550 8750
+	0    -1   -1   0
+$EndComp
+Connection ~ 11950 8750
+Wire Wire Line
+	11950 8750 11950 8850
+Wire Wire Line
+	6600 4350 6600 3650
+Wire Wire Line
+	6600 3650 8700 3650
+Wire Wire Line
+	8700 3650 8700 1000
+Wire Wire Line
+	8700 1000 9400 1000
+Wire Wire Line
+	6350 4350 6600 4350
+Wire Wire Line
+	6650 4450 6650 3700
+Wire Wire Line
+	6650 3700 8750 3700
+Wire Wire Line
+	8750 3700 8750 1100
+Wire Wire Line
+	8750 1100 9400 1100
+Wire Wire Line
+	6350 4450 6650 4450
+Wire Wire Line
+	6700 4550 6700 3750
+Wire Wire Line
+	6700 3750 8800 3750
+Wire Wire Line
+	8800 3750 8800 1200
+Wire Wire Line
+	8800 1200 9400 1200
+Wire Wire Line
+	6350 4550 6700 4550
+Wire Wire Line
+	6750 4650 6750 3800
+Wire Wire Line
+	6750 3800 8850 3800
+Wire Wire Line
+	8850 3800 8850 1300
+Wire Wire Line
+	8850 1300 9400 1300
+Wire Wire Line
+	6350 4650 6750 4650
+Wire Wire Line
+	6800 4750 6800 3850
+Wire Wire Line
+	6800 3850 8900 3850
+Wire Wire Line
+	8900 3850 8900 1400
+Wire Wire Line
+	8900 1400 9400 1400
+Wire Wire Line
+	6350 4750 6800 4750
+Wire Wire Line
+	6850 4850 6850 3900
+Wire Wire Line
+	6850 3900 8950 3900
+Wire Wire Line
+	8950 3900 8950 1500
+Wire Wire Line
+	8950 1500 9400 1500
+Wire Wire Line
+	6350 4850 6850 4850
+Wire Wire Line
+	6900 4950 6900 3950
+Wire Wire Line
+	6900 3950 9000 3950
+Wire Wire Line
+	9000 3950 9000 1600
+Wire Wire Line
+	9000 1600 9400 1600
+Wire Wire Line
+	6350 4950 6900 4950
+Wire Wire Line
+	6950 5150 6950 4000
+Wire Wire Line
+	6950 4000 9050 4000
+Wire Wire Line
+	9050 4000 9050 1700
+Wire Wire Line
+	9050 1700 9400 1700
+Wire Wire Line
+	6350 5150 6950 5150
+Wire Wire Line
+	9650 3950 9100 3950
+Wire Wire Line
+	9100 3950 9100 1800
+Wire Wire Line
+	9100 1800 9400 1800
+Wire Wire Line
+	9650 3950 9650 6250
+Wire Wire Line
+	9750 3900 9150 3900
+Wire Wire Line
+	9150 3900 9150 1900
+Wire Wire Line
+	9150 1900 9400 1900
+Wire Wire Line
+	9750 3900 9750 6350
+NoConn ~ 10500 4750
+NoConn ~ 10500 4850
+NoConn ~ 10500 4950
+NoConn ~ 10500 5050
+Wire Bus Line
+	3700 9250 3700 10150
+Wire Bus Line
+	1300 5050 1300 9050
+Wire Bus Line
+	5500 5350 5500 10150
+Wire Bus Line
+	3650 4250 3650 8000
 $EndSCHEMATC
